File: FPGA_AURA/FPGA_Power.kicad_sch (KiCad schematic)
At the start: 16 parts, among them U1 XC7A35T-2FTG256C

Commit message: Finished schematic to start routing again, and started MII fanout from connector.
Parts:
- renumbered C32 to C200, C18 to C201, C19 to C202, C20 to C203, C27 to C204, C26 to C205, C23 to C206, C21 to C207, C28 to C208, C25 to C209, C22 to C210, C24 to C211, C29 to C212, C30 to C213, C31 to C214
Other:
- company: (none) -> Alexander Armitage
- moved on the sheet: C200, C201, C202, C203, C204, C205, C206, C207, C208, C209, C210, C211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

Commit message: Schematic initial draft complete.
Parts:
- C200, C209: value 47 -> 47u
Changed lines of the file:
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@@
 			)
 		)
-		(property "Value" "47"
+		(property "Value" "47u"
 			(at 154.94 118.1099 0)
 			(show_name no)
@@
 			)
 		)
-		(property "Value" "47"
+		(property "Value" "47u"
 			(at 142.24 60.9599 0)
 			(show_name no)
