File: FPGA_AURA/Power_Regulation.kicad_sch (KiCad schematic)
At the start: 52 parts, among them U200 ADP5014, U4 TPS51200DRCR

Commit message: Finished schematic to start routing again, and started MII fanout from connector.
Parts:
- added H100, H101, H102, H103: MountingHole_Pad, MountingHole:MountingHole_3.2mm_M3_Pad_Via, symbol Mechanical:MountingHole_Pad
- renumbered C200 to C100, C201 to C101, C202 to C102, C203 to C103, C205 to C105, C206 to C106, C207 to C107, C208 to C108, C209 to C109, C210 to C110, C211 to C111, C212 to C112, C213 to C113, C214 to C114, C215 to C115, C216 to C116, C217 to C117, C218 to C118, C219 to C119, C220 to C120, C221 to C121, C222 to C122, L200 to L100, L201 to L101, L202 to L102, L203 to L103, R200 to R100, R201 to R101, R202 to R102, R203 to R103, R204 to R104, R205 to R105, R206 to R106, R207 to R107, R208 to R108, R209 to R109, R210 to R110, R211 to R111, R212 to R112, R213 to R113, R214 to R114, R215 to R115, R216 to R116, R217 to R117, R218 to R118, R219 to R119, R221 to R121, R222 to R122, R223 to R123, U200 to U100
Connections:
- net GND: now also H100.1, H101.1, H102.1, H103.1
Other:
- note removed: "ToDo: Validate component values Validate power up sequence"
- company: (none) -> Alexander Armitage
- moved on the sheet: C114, C115, C116, C117, C118, C119, C121, C122, R121, R122, R123, R220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

Commit message: Finishing off routing, fanning out fly by termination, and added ground pours
Connections:
- net +VREF: no longer C114.1, U4.6 (REFOUT)
- new net +VREF_DDR: C114.1, U4.6 (REFOUT)
Changed lines of the file:
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@@
 			)
 		)
-		(property "Value" "+VREF"
-			(at 257.81 63.5 0)
+		(property "Value" "+VREF_DDR"
+			(at 260.35 67.3099 0)
 			(show_name no)
 			(do_not_autoplace no)
@@
 					(size 1.27 1.27)
 				)
+				(justify left)
 			)
 		)
